File: hardware/tps62913-module.sch (KiCad schematic (older format))
At the start: 27 parts, among them J1 Conn_01x05, U1 TPS62913

Commit message: fix
Parts:
- C1, C10, C11, C12, C2, C3, C4, C5, C6, C7, C8, C9: Elecrow PN 302010103 -> (none); Original N -> (none); manf# CC0603KRX5R6BB106 -> (none)
- C13, C14: Elecrow PN 302010178 -> (none); Original N -> (none); manf# CC0805KKX5R8BB106 -> (none)
- C15: Elecrow PN 302010022 -> (none); Original N -> (none); manf# CC0402KRX7R9BB222 -> (none)
- C16: Elecrow PN 302010040 -> (none); Original N -> (none); manf# CC0402KRX5R6BB105 -> (none)
- FB1: Link https://www.mouser.jp/ProductDetail/Murata-Electronics/BLE1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 -> (none); Mouser # 81-BLE18PS080SN1D -> (none); Original Y -> (none)
- L1: Elecrow PN 303010103 -> (none); Original N -> (none); manf# SWPA5020S2R2NT -> (none)
- R1: Link https://www.mouser.jp/ProductDetail/YAGEO/RC0603FR-0742K2L?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 -> (none); Mouser # 603-RC0603FR-0742K2L -> (none); Original N -> (none); Rating Shenzhen stock -> (none); manf# RC0603FR-0742K2L -> (none)
- R2: Elecrow PN 301010254 -> (none); Original N -> (none); manf# RC0603FR-071K8L -> (none)
- R3: Elecrow PN 301010196 -> (none); manf# RC0603FR-07100KL -> (none)
- RV1: Elecrow PN 1051010A -> (none); manf# 3362P-1-103 -> (none)
- U1: Mouser # 595-TPS62913RPUR -> (none); Original Y -> (none)
